File: Power_Step Slave Board/Power_Step Slave Board.sch (KiCad schematic (older format))
At the start: 17 parts

Commit message: rev0.1
Parts:
- D1, D2: renamed from D?; footprint (none) -> LEDs:LED_D3.0mm
- P1, P10, P12, P13, P2, P5, P7, P9: renamed from P?; footprint Molex_KK_4x2.54mm_Straight -> Connectors_Molex:Molex_KK-6410-04_04x2.54mm_Straight
- R1, R2: renamed from R?; footprint (none) -> Resistors_ThroughHole:R_Axial_DIN0207_L6.3mm_D2.5mm_P7.62mm_Horizontal
- gave numbers to parts that had none: 5
Changed lines of the file:
@@
 $EndDescr
 $Comp
-L CONN_01X02 P?
+L CONN_01X02 P3
 U 1 1 59DE12D0
 P 2000 2750
-F 0 "P?" H 2000 2900 50  0000 C CNN
+F 0 "P3" H 2000 2900 50  0000 C CNN
 F 1 "CONN_01X02" V 2100 2750 50  0000 C CNN
 F 2 "ASSETS:CONN_ON_SHORE_2x_15A" H 2000 2750 50  0001 C CNN
@@
 $EndComp
 $Comp
-L CONN_01X02 P?
+L CONN_01X02 P6
 U 1 1 59DE1351
 P 3200 2750
-F 0 "P?" H 3200 2900 50  0000 C CNN
+F 0 "P6" H 3200 2900 50  0000 C CNN
 F 1 "CONN_01X02" V 3300 2750 50  0000 C CNN
 F 2 "ASSETS:CONN_ON_SHORE_2x_15A" H 3200 2750 50  0001 C BNN
@@
 $EndComp
 $Comp
-L CONN_01X02 P?
+L CONN_01X02 P4
 U 1 1 59DE13AE
 P 2700 3300
-F 0 "P?" H 2700 3450 50  0000 C CNN
+F 0 "P4" H 2700 3450 50  0000 C CNN
 F 1 "CONN_01X02" V 2800 3300 50  0000 C CNN
 F 2 "ASSETS:CONN_ON_SHORE_2x_15A" H 2700 3300 50  0001 C CNN
@@
 $EndComp
 $Comp
-L CONN_01X02 P?
+L CONN_01X02 P8
 U 1 1 59DE1578
 P 4200 2750
-F 0 "P?" H 4200 2900 50  0000 C CNN
+F 0 "P8" H 4200 2900 50  0000 C CNN
 F 1 "CONN_01X02" V 4300 2750 50  0000 C CNN
 F 2 "ASSETS:CONN_ON_SHORE_2x_15A" H 4200 2750 50  0001 C CNN
@@
 $EndComp
 $Comp
-L CONN_01X02 P?
+L CONN_01X02 P11
 U 1 1 59DE15C8
 P 5600 2750
-F 0 "P?" H 5600 2900 50  0000 C CNN
+F 0 "P11" H 5600 2900 50  0000 C CNN
 F 1 "CONN_01X02" V 5700 2750 50  0000 C CNN
 F 2 "ASSETS:CONN_ON_SHORE_2x_15A" H 5600 2750 50  0001 C CNN
@@
 $EndComp
 $Comp
-L CONN_01X04 P?
+L CONN_01X04 P1
 U 1 1 59E07C82
 P 1250 1450
-F 0 "P?" H 1250 1700 50  0000 C CNN
+F 0 "P1" H 1250 1700 50  0000 C CNN
 F 1 "CONN_01X04" V 1350 1450 50  0000 C CNN
-F 2 "Molex_KK_4x2.54mm_Straight" V 1450 1450 50  0000 C BNN
+F 2 "Connectors_Molex:Molex_KK-6410-04_04x2.54mm_Straight" V 1450 1450 50  0001 C BNN
 F 3 "" H 1250 1450 50  0000 C CNN
 	1    1250 1450
@@
 $EndComp
 $Comp
-L CONN_01X04 P?
+L CONN_01X04 P2
 U 1 1 59E07D10
 P 1900 1450
-F 0 "P?" H 1900 1700 50  0000 C CNN
+F 0 "P2" H 1900 1700 50  0000 C CNN
 F 1 "CONN_01X04" V 2000 1450 50  0000 C CNN
-F 2 "Molex_KK_4x2.54mm_Straight" V 2100 1450 50  0000 C CNN
+F 2 "Connectors_Molex:Molex_KK-6410-04_04x2.54mm_Straight" V 2100 1450 50  0001 C CNN
 F 3 "" H 1900 1450 50  0000 C CNN
 	1    1900 1450
@@
 $EndComp
 $Comp
-L CONN_01X04 P?
+L CONN_01X04 P5
 U 1 1 59E081DD
 P 2750 1450
-F 0 "P?" H 2750 1700 50  0000 C CNN
+F 0 "P5" H 2750 1700 50  0000 C CNN
 F 1 "CONN_01X04" V 2850 1450 50  0000 C CNN
-F 2 "Molex_KK_4x2.54mm_Straight" V 2950 1450 50  0000 C BNN
+F 2 "Connectors_Molex:Molex_KK-6410-04_04x2.54mm_Straight" V 2950 1450 50  0001 C BNN
 F 3 "" H 2750 1450 50  0000 C CNN
 	1    2750 1450
@@
 $EndComp
 $Comp
-L CONN_01X04 P?
+L CONN_01X04 P7
 U 1 1 59E081E3
 P 3400 1450
-F 0 "P?" H 3400 1700 50  0000 C CNN
+F 0 "P7" H 3400 1700 50  0000 C CNN
 F 1 "CONN_01X04" V 3500 1450 50  0000 C CNN
-F 2 "Molex_KK_4x2.54mm_Straight" V 3600 1450 50  0000 C CNN
+F 2 "Connectors_Molex:Molex_KK-6410-04_04x2.54mm_Straight" V 3600 1450 50  0001 C CNN
 F 3 "" H 3400 1450 50  0000 C CNN
 	1    3400 1450
@@
 $EndComp
 $Comp
-L CONN_01X04 P?
+L CONN_01X04 P9
 U 1 1 59E08812
 P 4350 1450
-F 0 "P?" H 4350 1700 50  0000 C CNN
+F 0 "P9" H 4350 1700 50  0000 C CNN
 F 1 "CONN_01X04" V 4450 1450 50  0000 C CNN
-F 2 "Molex_KK_4x2.54mm_Straight" V 4550 1450 50  0000 C BNN
+F 2 "Connectors_Molex:Molex_KK-6410-04_04x2.54mm_Straight" V 4550 1450 50  0001 C BNN
 F 3 "" H 4350 1450 50  0000 C CNN
 	1    4350 1450
@@
 $EndComp
 $Comp
-L CONN_01X04 P?
+L CONN_01X04 P10
 U 1 1 59E08818
 P 5000 1450
-F 0 "P?" H 5000 1700 50  0000 C CNN
+F 0 "P10" H 5000 1700 50  0000 C CNN
 F 1 "CONN_01X04" V 5100 1450 50  0000 C CNN
-F 2 "Molex_KK_4x2.54mm_Straight" V 5200 1450 50  0000 C CNN
+F 2 "Connectors_Molex:Molex_KK-6410-04_04x2.54mm_Straight" V 5200 1450 50  0001 C CNN
 F 3 "" H 5000 1450 50  0000 C CNN
 	1    5000 1450
@@
 $EndComp
 $Comp
-L CONN_01X04 P?
+L CONN_01X04 P12
 U 1 1 59E08822
 P 5850 1450
-F 0 "P?" H 5850 1700 50  0000 C CNN
+F 0 "P12" H 5850 1700 50  0000 C CNN
 F 1 "CONN_01X04" V 5950 1450 50  0000 C CNN
-F 2 "Molex_KK_4x2.54mm_Straight" V 6050 1450 50  0000 C BNN
+F 2 "Connectors_Molex:Molex_KK-6410-04_04x2.54mm_Straight" V 6050 1450 50  0001 C BNN
 F 3 "" H 5850 1450 50  0000 C CNN
 	1    5850 1450
@@
 $EndComp
 $Comp
-L CONN_01X04 P?
+L CONN_01X04 P13
 U 1 1 59E08828
 P 6500 1450
-F 0 "P?" H 6500 1700 50  0000 C CNN
+F 0 "P13" H 6500 1700 50  0000 C CNN
 F 1 "CONN_01X04" V 6600 1450 50  0000 C CNN
-F 2 "Molex_KK_4x2.54mm_Straight" V 6700 1450 50  0000 C CNN
+F 2 "Connectors_Molex:Molex_KK-6410-04_04x2.54mm_Straight" V 6700 1450 50  0001 C CNN
 F 3 "" H 6500 1450 50  0000 C CNN
 	1    6500 1450
@@
 $EndComp
 $Comp
-L R R?
+L R R1
 U 1 1 59E0902D
 P 2200 2300
-F 0 "R?" V 2280 2300 50  0000 C CNN
+F 0 "R1" V 2280 2300 50  0000 C CNN
 F 1 "R" V 2200 2300 50  0000 C CNN
-F 2 "" V 2130 2300 50  0000 C CNN
+F 2 "Resistors_ThroughHole:R_Axial_DIN0207_L6.3mm_D2.5mm_P7.62mm_Horizontal" V 2130 2300 50  0001 C CNN
 F 3 "" H 2200 2300 50  0000 C CNN
 	1    2200 2300
@@
 $EndComp
 $Comp
-L LED D?
+L LED D1
 U 1 1 59E0909A
 P 2650 2300
-F 0 "D?" H 2650 2400 50  0000 C CNN
+F 0 "D1" H 2650 2400 50  0000 C CNN
 F 1 "LED" H 2650 2200 50  0000 C CNN
-F 2 "" H 2650 2300 50  0000 C CNN
+F 2 "LEDs:LED_D3.0mm" H 2650 2300 50  0001 C CNN
 F 3 "" H 2650 2300 50  0000 C CNN
 	1    2650 2300
@@
 $EndComp
 $Comp
-L R R?
+L R R2
 U 1 1 59E098E0
 P 4650 2300
-F 0 "R?" V 4730 2300 50  0000 C CNN
+F 0 "R2" V 4730 2300 50  0000 C CNN
 F 1 "R" V 4650 2300 50  0000 C CNN
-F 2 "" V 4580 2300 50  0000 C CNN
+F 2 "Resistors_ThroughHole:R_Axial_DIN0207_L6.3mm_D2.5mm_P7.62mm_Horizontal" V 4580 2300 50  0001 C CNN
 F 3 "" H 4650 2300 50  0000 C CNN
 	1    4650 2300
@@
 $EndComp
 $Comp
-L LED D?
+L LED D2
 U 1 1 59E098E6
 P 5050 2300
-F 0 "D?" H 5050 2400 50  0000 C CNN
+F 0 "D2" H 5050 2400 50  0000 C CNN
 F 1 "LED" H 5050 2200 50  0000 C CNN
-F 2 "" H 5050 2300 50  0000 C CNN
+F 2 "LEDs:LED_D3.0mm" H 5050 2300 50  0001 C CNN
 F 3 "" H 5050 2300 50  0000 C CNN
 	1    5050 2300

Commit message: created PCB
Parts:
- added D3: LED, LEDs:LED_D3.0mm, symbol LED
- added R3: R, Resistors_ThroughHole:R_Axial_DIN0207_L6.3mm_D2.5mm_P7.62mm_Horizontal, symbol R
Connections:
- net at D1.1 (K), P3.1 (P1), P4.1 (P1)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: now also D3.1 (K)
- net at P3.2 (P2), P4.2 (P2), P6.2 (P2)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: now also R3.2
- new net: D3.2 (A), R3.1
Changed lines of the file:
@@
 	2350 2300 2450 2300
 Wire Wire Line
-	2850 2300 2850 2700
+	2850 2050 2850 2700
 Connection ~ 2850 2700
 Wire Wire Line
 	2050 2300 1800 2300
 Wire Wire Line
-	1800 2300 1800 3350
+	1800 2050 1800 3350
 Connection ~ 2350 3350
 Wire Wire Line
@@
 	5250 2300 5250 2700
 Connection ~ 5250 2700
+$Comp
+L R R3
+U 1 1 59E0AF44
+P 2200 2050
+F 0 "R3" V 2280 2050 50  0000 C CNN
+F 1 "R" V 2200 2050 50  0000 C CNN
+F 2 "Resistors_ThroughHole:R_Axial_DIN0207_L6.3mm_D2.5mm_P7.62mm_Horizontal" V 2130 2050 50  0001 C CNN
+F 3 "" H 2200 2050 50  0000 C CNN
+	1    2200 2050
+	0    1    1    0
+$EndComp
+$Comp
+L LED D3
+U 1 1 59E0AF4A
+P 2650 2050
+F 0 "D3" H 2650 2150 50  0000 C CNN
+F 1 "LED" H 2650 1950 50  0000 C CNN
+F 2 "LEDs:LED_D3.0mm" H 2650 2050 50  0001 C CNN
+F 3 "" H 2650 2050 50  0000 C CNN
+	1    2650 2050
+	-1   0    0    1
+$EndComp
+Wire Wire Line
+	2350 2050 2450 2050
+Wire Wire Line
+	2050 2050 1800 2050
+Connection ~ 1800 2300
+Connection ~ 2850 2300
 $EndSCHEMATC

Commit message: Next rev
Parts:
- D1, D3: footprint LEDs:LED_D3.0mm -> LEDs:LED_0603
- R1, R3: footprint Resistors_ThroughHole:R_Axial_DIN0207_L6.3mm_D2.5mm_P7.62mm_Horizontal -> Resistors_SMD:R_0603
Connections:
- net GND: now reaches D1.1 (K), D3.1 (K), P3.1 (P1), P4.1 (P1), P6.1 (P1)
- net GND: now also D2.1 (K), P11.1 (P1), P8.1 (P1)
Changed lines of the file:
@@
 F 0 "R1" V 2280 2300 50  0000 C CNN
 F 1 "R" V 2200 2300 50  0000 C CNN
-F 2 "Resistors_ThroughHole:R_Axial_DIN0207_L6.3mm_D2.5mm_P7.62mm_Horizontal" V 2130 2300 50  0001 C CNN
+F 2 "Resistors_SMD:R_0603" V 2130 2300 50  0001 C CNN
 F 3 "" H 2200 2300 50  0000 C CNN
 	1    2200 2300
@@
 F 0 "D1" H 2650 2400 50  0000 C CNN
 F 1 "LED" H 2650 2200 50  0000 C CNN
-F 2 "LEDs:LED_D3.0mm" H 2650 2300 50  0001 C CNN
+F 2 "LEDs:LED_0603" H 2650 2300 50  0001 C CNN
 F 3 "" H 2650 2300 50  0000 C CNN
 	1    2650 2300
@@
 	1    5050 2300
 	-1   0    0    1
+$EndComp
+$Comp
+L R R3
+U 1 1 59E0AF44
+P 2200 2050
+F 0 "R3" V 2280 2050 50  0000 C CNN
+F 1 "R" V 2200 2050 50  0000 C CNN
+F 2 "Resistors_SMD:R_0603" V 2130 2050 50  0001 C CNN
+F 3 "" H 2200 2050 50  0000 C CNN
+	1    2200 2050
+	0    1    1    0
+$EndComp
+$Comp
+L LED D3
+U 1 1 59E0AF4A
+P 2650 2050
+F 0 "D3" H 2650 2150 50  0000 C CNN
+F 1 "LED" H 2650 1950 50  0000 C CNN
+F 2 "LEDs:LED_0603" H 2650 2050 50  0001 C CNN
+F 3 "" H 2650 2050 50  0000 C CNN
+	1    2650 2050
+	-1   0    0    1
+$EndComp
+$Comp
+L GND #PWR01
+U 1 1 59E204D5
+P 3050 2300
+F 0 "#PWR01" H 3050 2050 50  0001 C CNN
+F 1 "GND" H 3050 2150 50  0000 C CNN
+F 2 "" H 3050 2300 50  0000 C CNN
+F 3 "" H 3050 2300 50  0000 C CNN
+	1    3050 2300
+	1    0    0    -1
+$EndComp
+$Comp
+L GND #PWR02
+U 1 1 59E2050F
+P 5400 2450
+F 0 "#PWR02" H 5400 2200 50  0001 C CNN
+F 1 "GND" H 5400 2300 50  0000 C CNN
+F 2 "" H 5400 2450 50  0000 C CNN
+F 3 "" H 5400 2450 50  0000 C CNN
+	1    5400 2450
+	1    0    0    -1
 $EndComp
 Wire Wire Line
@@
 	5250 2300 5250 2700
 Connection ~ 5250 2700
-$Comp
-L R R3
-U 1 1 59E0AF44
-P 2200 2050
-F 0 "R3" V 2280 2050 50  0000 C CNN
-F 1 "R" V 2200 2050 50  0000 C CNN
-F 2 "Resistors_ThroughHole:R_Axial_DIN0207_L6.3mm_D2.5mm_P7.62mm_Horizontal" V 2130 2050 50  0001 C CNN
-F 3 "" H 2200 2050 50  0000 C CNN
-	1    2200 2050
-	0    1    1    0
-$EndComp
-$Comp
-L LED D3
-U 1 1 59E0AF4A
-P 2650 2050
-F 0 "D3" H 2650 2150 50  0000 C CNN
-F 1 "LED" H 2650 1950 50  0000 C CNN
-F 2 "LEDs:LED_D3.0mm" H 2650 2050 50  0001 C CNN
-F 3 "" H 2650 2050 50  0000 C CNN
-	1    2650 2050
-	-1   0    0    1
-$EndComp
 Wire Wire Line
 	2350 2050 2450 2050
@@
 Connection ~ 1800 2300
 Connection ~ 2850 2300
+Wire Wire Line
+	5400 2450 5250 2450
+Connection ~ 5250 2450
+Wire Wire Line
+	2850 2300 3050 2300
 $EndSCHEMATC
