File: Power_Step Slave Board/Power_Step Slave Board.kicad_pcb (KiCad board)
At the start: 2 copper layers, 17 parts, among them P1 CONN_01X04, P10 CONN_01X04, P11 CONN_01X02, P12 CONN_01X04, P13 CONN_01X04, P2 CONN_01X04, P3 CONN_01X02, P4 CONN_01X02, P5 CONN_01X04, P6 CONN_01X02, P7 CONN_01X04, P8 CONN_01X02, P9 CONN_01X04

Commit message: created PCB
Parts:
- added D3: LED, LEDs:LED_D3.0mm, F.Cu at (160.0, 111.8)
- added R3: R, Resistors_ThroughHole:R_Axial_DIN0207_L6.3mm_D2.5mm_P7.62mm_Horizontal, F.Cu at (153.7, 115.6)
- P1, P12, P13, P5, P7, P9: moved to B.Cu
- P3: moved to F.Cu
- moved D2 54.6 mm to (144.8, 87.6)
- moved R1 48.6 mm to (151.1, 96.5), turned to 270 degrees
- moved P6 48.5 mm to (129.5, 110.5), turned to 270 degrees
- moved R2 47.1 mm to (135.9, 83.8)
- moved P5 43.1 mm to (153.7, 127.0), turned to 90 degrees
- moved P11 42.3 mm to (151.1, 86.4), turned to 90 degrees
- moved D1 41.5 mm to (157.5, 99.1), turned to 180 degrees
- moved P12 40.5 mm to (168.9, 127.0), turned to 90 degrees
- moved P1 34.2 mm to (127.0, 127.0), turned to 90 degrees
- moved P7 28.2 mm to (146.1, 127.0), turned to 90 degrees
- moved P8 27.9 mm to (132.1, 96.5), turned to 270 degrees
- moved P13 25.2 mm to (161.3, 127.0), turned to 90 degrees
- moved P2 24.5 mm to (144.8, 102.9), turned to 90 degrees
- moved P4 18.1 mm to (166.4, 111.8), turned to 90 degrees
- moved P3 16.7 mm to (163.8, 99.1), turned to 90 degrees
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Other:
- board outline added: 69.4 x 49.1 mm

Commit message: Next rev
Parts:
- D1, D2, D3: footprint LEDs:LED_D3.0mm -> LEDs:LED_0603
- R1, R2, R3: footprint Resistors_ThroughHole:R_Axial_DIN0207_L6.3mm_D2.5mm_P7.62mm_Horizontal -> Resistors_SMD:R_0603
- moved R1 9.25 mm to (160.0, 99.1), turned to 90 degrees
- moved R3 9.17 mm to (162.2, 112.1)
- moved P10 8.44 mm to (149.4, 108.2), turned to 180 degrees
- moved P11 7.49 mm to (143.6, 86.5)
- moved P2 6.65 mm to (149.4, 98.0), turned to 180 degrees
- moved R2 6.30 mm to (140.6, 88.0), turned to 90 degrees
- moved D2 5.34 mm to (140.6, 90.9), turned to 90 degrees
- moved D1 4.58 mm to (160.0, 102.9), turned to 90 degrees
- moved D3 4.27 mm to (162.2, 115.4), turned to 90 degrees
- moved P13 2.16 mm to (163.4, 127.0)
- moved P5 2.16 mm to (155.8, 127.0)
- moved P12 2.16 mm to (171.1, 127.0)
- moved P7 2.16 mm to (148.2, 127.0)
- moved P8 2.03 mm to (132.1, 94.5)
- moved P6 1.85 mm to (130.0, 108.7)
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Connections:
- D1 pad 1: Net-(D1-Pad1) -> GND
- D2 pad 1: Net-(D2-Pad1) -> GND
- D3 pad 1: Net-(D1-Pad1) -> GND
- P11 pad 1: Net-(D2-Pad1) -> GND
- P3 pad 1: Net-(D1-Pad1) -> GND
- P4 pad 1: Net-(D1-Pad1) -> GND
- P6 pad 1: Net-(D1-Pad1) -> GND
- P8 pad 1: Net-(D2-Pad1) -> GND
Routing:
- net Net-(P3-Pad2): track 0.00 -> 68.3 mm, vias 0 -> 2
- net Net-(P1-Pad1): track 0.00 -> 46.7 mm
- net Net-(P1-Pad3): track 0.00 -> 44.0 mm
- net Net-(P1-Pad2): track 0.00 -> 41.3 mm
- net Net-(P1-Pad4): track 0.00 -> 40.2 mm
- net Net-(P10-Pad1): track 0.00 -> 28.8 mm
- net Net-(P11-Pad2): track 0.00 -> 28.7 mm
- net Net-(P10-Pad2): track 0.00 -> 23.7 mm
- net Net-(P10-Pad3): track 0.00 -> 18.2 mm
- net Net-(P10-Pad4): track 0.00 -> 13.6 mm
- net Net-(P5-Pad4): track 0.00 -> 7.62 mm
- net Net-(P5-Pad3): track 0.00 -> 7.62 mm
- net Net-(P5-Pad2): track 0.00 -> 7.62 mm
- net Net-(P5-Pad1): track 0.00 -> 7.62 mm
- net Net-(P12-Pad4): track 0.00 -> 7.62 mm
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- added copper zone on B.Cu, net GND
Other:
- net class STEPPER added: clearance 0.2, trace_width 1.5, via_dia 0.6, via_drill 0.4
- net class WIDE TRACK added: clearance 0.2, trace_width 5, via_dia 0.6, via_drill 0.4

Commit message: REV 0.1
Other:
- board text added: "24V - 10A MAX (Combined)"
- board text added: "4 AXIS"
- board text added: "5 AXIS"
- board text added: "5A MAX 24V"
- board text added: "Evezor Power/Step Distribution Board Rev 0.1"
- board text added: "TH"
Changed lines of the file:
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@@
     (area 113.74941 80.408997 183.252791 129.598203)
     (thickness 1.6)
-    (drawings 10)
+    (drawings 17)
     (tracks 99)
     (zones 0)
@@
   (layers
     (0 F.Cu signal)
-    (31 B.Cu signal)
+    (31 B.Cu signal hide)
     (32 B.Adhes user)
     (33 F.Adhes user)
@@
     (descr "Connector Headers with Friction Lock, 22-27-2041, http://www.molex.com/pdm_docs/sd/022272021_sd.pdf")
     (tags "connector molex kk_6410 22-27-2041")
-    (fp_text reference P1 (at 1 4.5 90) (layer B.SilkS)
+    (fp_text reference P1 (at 10.287 0.381 180) (layer B.SilkS)
       (effects (font (size 1 1) (thickness 0.15)) (justify mirror))
     )
@@
     (descr "Connector Headers with Friction Lock, 22-27-2041, http://www.molex.com/pdm_docs/sd/022272021_sd.pdf")
     (tags "connector molex kk_6410 22-27-2041")
-    (fp_text reference P2 (at 1 -4.5 180) (layer F.SilkS)
-      (effects (font (size 1 1) (thickness 0.15)))
+    (fp_text reference P2 (at 9.906 0 270) (layer F.SilkS)
+      (effects (font (size 0.5 0.5) (thickness 0.125)))
     )
     (fp_text value CONN_01X04 (at 3.81 4.5 180) (layer F.Fab)
@@
     (descr "Connector Headers with Friction Lock, 22-27-2041, http://www.molex.com/pdm_docs/sd/022272021_sd.pdf")
     (tags "connector molex kk_6410 22-27-2041")
-    (fp_text reference P5 (at 1 4.5 90) (layer B.SilkS)
+    (fp_text reference P5 (at 10.287 0.254 180) (layer B.SilkS)
       (effects (font (size 1 1) (thickness 0.15)) (justify mirror))
     )
@@
     (descr "Connector Headers with Friction Lock, 22-27-2041, http://www.molex.com/pdm_docs/sd/022272021_sd.pdf")
     (tags "connector molex kk_6410 22-27-2041")
-    (fp_text reference P7 (at 1 4.5 90) (layer B.SilkS)
+    (fp_text reference P7 (at 10.287 0.254 180) (layer B.SilkS)
       (effects (font (size 1 1) (thickness 0.15)) (justify mirror))
     )
@@
     (descr "Connector Headers with Friction Lock, 22-27-2041, http://www.molex.com/pdm_docs/sd/022272021_sd.pdf")
     (tags "connector molex kk_6410 22-27-2041")
-    (fp_text reference P9 (at 1 4.5 90) (layer B.SilkS)
+    (fp_text reference P9 (at 10.414 0.127 180) (layer B.SilkS)
       (effects (font (size 1 1) (thickness 0.15)) (justify mirror))
     )
@@
     (descr "Connector Headers with Friction Lock, 22-27-2041, http://www.molex.com/pdm_docs/sd/022272021_sd.pdf")
     (tags "connector molex kk_6410 22-27-2041")
-    (fp_text reference P10 (at 1 -4.5 180) (layer F.SilkS)
-      (effects (font (size 1 1) (thickness 0.15)))
+    (fp_text reference P10 (at 9.906 -0.127 270) (layer F.SilkS)
+      (effects (font (size 0.5 0.5) (thickness 0.125)))
     )
     (fp_text value CONN_01X04 (at 3.81 4.5 180) (layer F.Fab)
@@
     (descr "Connector Headers with Friction Lock, 22-27-2041, http://www.molex.com/pdm_docs/sd/022272021_sd.pdf")
     (tags "connector molex kk_6410 22-27-2041")
-    (fp_text reference P12 (at 1 4.5 90) (layer B.SilkS)
+    (fp_text reference P12 (at 10.287 0 180) (layer B.SilkS)
       (effects (font (size 1 1) (thickness 0.15)) (justify mirror))
     )
@@
     (descr "Connector Headers with Friction Lock, 22-27-2041, http://www.molex.com/pdm_docs/sd/022272021_sd.pdf")
     (tags "connector molex kk_6410 22-27-2041")
-    (fp_text reference P13 (at 1 4.5 90) (layer B.SilkS)
+    (fp_text reference P13 (at 10.16 -0.254 180) (layer B.SilkS)
       (effects (font (size 1 1) (thickness 0.15)) (justify mirror))
     )
@@
   (module ASSETS:CONN_ON_SHORE_2x_15A (layer F.Cu)
     (at 132.08 94.488 270)
-    (fp_text reference P8 (at 0.508 12.596 270) (layer F.SilkS)
+    (fp_text reference P8 (at 0.254 4.445 360) (layer F.SilkS)
       (effects (font (size 1 1) (thickness 0.15)))
     )
@@
   (module ASSETS:CONN_ON_SHORE_2x_15A (layer F.Cu)
     (at 163.83 99.06 90)
-    (fp_text reference P3 (at 0.508 12.596 90) (layer F.SilkS)
+    (fp_text reference P3 (at 0.127 4.953 180) (layer F.SilkS)
       (effects (font (size 1 1) (thickness 0.15)))
     )
@@
   (module ASSETS:CONN_ON_SHORE_2x_15A (layer F.Cu)
     (at 130.048 108.712 270)
-    (fp_text reference P6 (at 0.508 12.596 270) (layer F.SilkS)
+    (fp_text reference P6 (at 0.381 3.683 360) (layer F.SilkS)
       (effects (font (size 1 1) (thickness 0.15)))
     )
@@
   (module ASSETS:CONN_ON_SHORE_2x_15A (layer F.Cu)
     (at 165.608 111.633 90)
-    (fp_text reference P4 (at 0.508 12.596 90) (layer F.SilkS)
+    (fp_text reference P4 (at 0.127 4.445 180) (layer F.SilkS)
       (effects (font (size 1 1) (thickness 0.15)))
     )
@@
     (tags "LED led 0603 SMD smd SMT smt smdled SMDLED smtled SMTLED")
     (attr smd)
-    (fp_text reference D1 (at 0 -1.25 90) (layer F.SilkS)
-      (effects (font (size 1 1) (thickness 0.15)))
+    (fp_text reference D1 (at -1.905 0 180) (layer F.SilkS)
+      (effects (font (size 0.5 0.5) (thickness 0.125)))
     )
     (fp_text value LED (at 0 1.35 90) (layer F.Fab)
@@
     (attr smd)
     (fp_text reference D2 (at 0 -1.25 90) (layer F.SilkS)
-      (effects (font (size 1 1) (thickness 0.15)))
+      (effects (font (size 0.5 0.5) (thickness 0.125)))
     )
     (fp_text value LED (at 0 1.35 90) (layer F.Fab)
@@
     (tags "LED led 0603 SMD smd SMT smt smdled SMDLED smtled SMTLED")
     (attr smd)
-    (fp_text reference D3 (at 0 -1.25 90) (layer F.SilkS)
-      (effects (font (size 1 1) (thickness 0.15)))
+    (fp_text reference D3 (at -1.905 0 180) (layer F.SilkS)
+      (effects (font (size 0.5 0.5) (thickness 0.125)))
     )
     (fp_text value LED (at 0 1.35 90) (layer F.Fab)
@@
     (tags "resistor 0603")
     (attr smd)
-    (fp_text reference R2 (at 0 -1.45 90) (layer F.SilkS)
-      (effects (font (size 1 1) (thickness 0.15)))
+    (fp_text reference R2 (at 0 -1.143 90) (layer F.SilkS)
+      (effects (font (size 0.5 0.5) (thickness 0.125)))
     )
     (fp_text value R (at 0 1.5 90) (layer F.Fab)
@@
     (tags "resistor 0603")
     (attr smd)
-    (fp_text reference R3 (at 0 -1.45 90) (layer F.SilkS)
-      (effects (font (size 1 1) (thickness 0.15)))
+    (fp_text reference R3 (at 1.651 0 180) (layer F.SilkS)
+      (effects (font (size 0.5 0.5) (thickness 0.125)))
     )
     (fp_text value R (at 0 1.5 90) (layer F.Fab)
@@
     (tags "resistor 0603")
     (attr smd)
-    (fp_text reference R1 (at 0 -1.45 90) (layer F.SilkS)
-      (effects (font (size 1 1) (thickness 0.15)))
+    (fp_text reference R1 (at 1.651 0 180) (layer F.SilkS)
+      (effects (font (size 0.5 0.5) (thickness 0.125)))
     )
     (fp_text value R (at 0 1.5 90) (layer F.Fab)
@@
       (rotate (xyz 0 0 0))
     )
+  )
+  (gr_text TH (at 143.637 112.268) (layer F.SilkS)
+    (effects (font (size 0.5 0.5) (thickness 0.125)))
+  )
+  (gr_text TH (at 143.891 102.235) (layer F.SilkS)
+    (effects (font (size 0.5 0.5) (thickness 0.125)))
+  )
+  (gr_text "5 AXIS" (at 145.415 113.03) (layer F.SilkS)
+    (effects (font (size 1.5 1.5) (thickness 0.3)))
+  )
+  (gr_text "4 AXIS" (at 145.542 102.997) (layer F.SilkS)
+    (effects (font (size 1.5 1.5) (thickness 0.3)))
+  )
+  (gr_text "5A MAX\n24V" (at 161.798 86.233 90) (layer F.SilkS)
+    (effects (font (size 1.5 1.5) (thickness 0.3)))
+  )
+  (gr_text "24V - 10A MAX\n(Combined)" (at 155.067 107.188 90) (layer F.SilkS)
+    (effects (font (size 1.5 1.5) (thickness 0.3)))
+  )
+  (gr_text "Evezor Power/Step \nDistribution Board Rev 0.1" (at 127.889 116.586) (layer F.SilkS)
+    (effects (font (size 0.75 0.75) (thickness 0.1875)))
   )
   (gr_circle (center 167.763414 83.85427) (end 169.263414 83.85427) (layer Edge.Cuts) (width 0.1))
@@
     (polygon
       (pts
-        (xy 119.888 117.856) (xy 127.127 80.645) (xy 169.926 80.645) (xy 177.165 118.11)
+        (xy 118.11 129.54) (xy 127.127 80.645) (xy 169.926 80.645) (xy 179.07 129.54)
       )
     )

Commit message: routing fixes
Parts:
- added REF**: MountingHole_3.2mm_M3, Mounting_Holes:MountingHole_3.2mm_M3, F.Cu at (129.2, 83.9)
- added REF**: MountingHole_3.2mm_M3, Mounting_Holes:MountingHole_3.2mm_M3, F.Cu at (167.7, 83.9)
- added REF**: MountingHole_3.2mm_M3, Mounting_Holes:MountingHole_3.2mm_M3, F.Cu at (118.4, 125.1)
- added REF**: MountingHole_3.2mm_M3, Mounting_Holes:MountingHole_3.2mm_M3, F.Cu at (178.6, 125.1)
- moved P10 0.76 mm to (150.1, 108.3)
Routing:
- net GND: track 6.18 -> 13.4 mm, vias 3 -> 0
- net Net-(P1-Pad1): track 46.7 -> 41.8 mm
- net Net-(P3-Pad2): track 68.3 -> 63.6 mm, vias 2 -> 0
- net Net-(P10-Pad1): track 28.8 -> 24.2 mm
- net Net-(P1-Pad4): track 40.2 -> 35.9 mm
- net Net-(P1-Pad2): track 41.3 -> 38.1 mm
- net Net-(P10-Pad2): track 23.7 -> 20.6 mm
- net Net-(P1-Pad3): track 44.0 -> 42.5 mm
- net Net-(P10-Pad3): track 18.2 -> 17.1 mm
- net Net-(P11-Pad2): track 28.7 -> 29.4 mm
Other:
- outline, holes or cut-outs redrawn

Commit message: more fixes
Routing:
- net Net-(P11-Pad2): track 29.4 -> 20.7 mm
Changed lines of the file:
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@@
     (thickness 1.6)
     (drawings 13)
-    (tracks 92)
+    (tracks 88)
     (zones 0)
     (modules 23)
@@
     (add_net "Net-(D2-Pad2)")
     (add_net "Net-(D3-Pad2)")
-    (add_net "Net-(P11-Pad2)")
     (add_net "Net-(P3-Pad2)")
   )
@@
     (uvia_dia 0.3)
     (uvia_drill 0.1)
+    (add_net "Net-(P11-Pad2)")
   )
   (module Connectors_Molex:Molex_KK-6410-04_04x2.54mm_Straight (layer F.Cu)
@@
   (segment (start 160.02 102.07) (end 160.02 99.81) (width 0.25) (layer F.Cu) (net 1))
   (segment (start 140.589 90.132) (end 140.589 88.761) (width 0.25) (layer F.Cu) (net 2))
+  (segment (start 142.748 104.0892) (end 146.1068 104.0892) (width 1.5) (layer F.Cu) (net 3))
   (segment (start 127 127) (end 129.8 127) (width 1.5) (layer F.Cu) (net 3))
-  (segment (start 129.8 127) (end 134.62 122.18) (width 1.5) (layer F.Cu) (net 3))
+  (segment (start 129.8 127) (end 134.948411 121.851589) (width 1.5) (layer F.Cu) (net 3))
+  (segment (start 134.948411 111.888789) (end 142.748 104.0892) (width 1.5) (layer F.Cu) (net 3))
+  (segment (start 134.948411 121.851589) (end 134.948411 111.888789) (width 1.5) (layer F.Cu) (net 3))
+  (segment (start 146.1068 104.0892) (end 149.352 100.844) (width 1.5) (layer F.Cu) (net 3))
   (segment (start 149.352 100.844) (end 149.352 98.044) (width 1.5) (layer F.Cu) (net 3))
-  (segment (start 134.62 122.18) (end 134.62 112.25827) (width 1.5) (layer F.Cu) (net 3))
-  (segment (start 134.62 112.25827) (end 142.78907 104.0892) (width 1.5) (layer F.Cu) (net 3))
-  (segment (start 142.78907 104.0892) (end 146.1068 104.0892) (width 1.5) (layer F.Cu) (net 3))
-  (segment (start 146.1068 104.0892) (end 149.352 100.844) (width 1.5) (layer F.Cu) (net 3))
-  (segment (start 145.4464 102.2096) (end 146.812 100.844) (width 1.5) (layer F.Cu) (net 4))
   (segment (start 127 124.46) (end 129.8 124.46) (width 1.5) (layer F.Cu) (net 4))
   (segment (start 146.812 100.844) (end 146.812 98.044) (width 1.5) (layer F.Cu) (net 4))
-  (segment (start 132.588 111.886092) (end 142.264492 102.2096) (width 1.5) (layer F.Cu) (net 4))
-  (segment (start 129.8 124.46) (end 132.588 121.672) (width 1.5) (layer F.Cu) (net 4))
-  (segment (start 132.588 121.672) (end 132.588 111.886092) (width 1.5) (layer F.Cu) (net 4))
-  (segment (start 142.264492 102.2096) (end 145.4464 102.2096) (width 1.5) (layer F.Cu) (net 4))
+  (segment (start 133.248401 111.184621) (end 142.043833 102.389189) (width 1.5) (layer F.Cu) (net 4))
+  (segment (start 133.2484 121.0116) (end 133.248401 111.184621) (width 1.5) (layer F.Cu) (net 4))
+  (segment (start 129.8 124.46) (end 133.2484 121.0116) (width 1.5) (layer F.Cu) (net 4))
+  (segment (start 142.043833 102.389189) (end 145.266811 102.389189) (width 1.5) (layer F.Cu) (net 4))
+  (segment (start 145.266811 102.389189) (end 146.812 100.844) (width 1.5) (layer F.Cu) (net 4))
+  (segment (start 129.8 121.92) (end 130.1496 121.5704) (width 1.5) (layer F.Cu) (net 5))
   (segment (start 144.272 98.56173) (end 144.272 98.044) (width 1.5) (layer F.Cu) (net 5))
-  (segment (start 141.775904 100.29401) (end 142.53972 100.29401) (width 1.5) (layer F.Cu) (net 5))
-  (segment (start 129.032 102.2604) (end 139.809514 102.2604) (width 1.5) (layer F.Cu) (net 5))
+  (segment (start 142.144552 100.689178) (end 144.272 98.56173) (width 1.5) (layer F.Cu) (net 5))
+  (segment (start 141.339666 100.689178) (end 142.144552 100.689178) (width 1.5) (layer F.Cu) (net 5))
   (segment (start 126.414011 104.878389) (end 129.032 102.2604) (width 1.5) (layer F.Cu) (net 5))
   (segment (start 126.414011 114.171211) (end 126.414011 104.878389) (width 1.5) (layer F.Cu) (net 5))
+  (segment (start 139.768444 102.2604) (end 141.339666 100.689178) (width 1.5) (layer F.Cu) (net 5))
+  (segment (start 129.032 102.2604) (end 139.768444 102.2604) (width 1.5) (layer F.Cu) (net 5))
   (segment (start 130.1496 117.9068) (end 126.414011 114.171211) (width 1.5) (layer F.Cu) (net 5))
+  (segment (start 127 121.92) (end 129.8 121.92) (width 1.5) (layer F.Cu) (net 5))
   (segment (start 130.1496 121.5704) (end 130.1496 117.9068) (width 1.5) (layer F.Cu) (net 5))
-  (segment (start 127 121.92) (end 129.8 121.92) (width 1.5) (layer F.Cu) (net 5))
-  (segment (start 129.8 121.92) (end 130.1496 121.5704) (width 1.5) (layer F.Cu) (net 5))
-  (segment (start 142.53972 100.29401) (end 144.272 98.56173) (width 1.5) (layer F.Cu) (net 5))
-  (segment (start 139.809514 102.2604) (end 141.775904 100.29401) (width 1.5) (layer F.Cu) (net 5))
-  (segment (start 128.327833 100.560389) (end 124.714 104.174222) (width 1.5) (layer F.Cu) (net 6))
-  (segment (start 139.105347 100.560389) (end 128.327833 100.560389) (width 1.5) (layer F.Cu) (net 6))
-  (segment (start 141.732 98.044) (end 141.621736 98.044) (width 1.5) (layer F.Cu) (net 6))
-  (segment (start 141.621736 98.044) (end 139.105347 100.560389) (width 1.5) (layer F.Cu) (net 6))
-  (segment (start 124.714 104.174222) (end 124.714 117.394) (width 1.5) (layer F.Cu) (net 6))
-  (segment (start 124.714 117.394) (end 126.7 119.38) (width 1.5) (layer F.Cu) (net 6))
+  (segment (start 139.064277 100.560389) (end 128.327833 100.560389) (width 1.5) (layer F.Cu) (net 6))
+  (segment (start 141.732 98.044) (end 141.580666 98.044) (width 1.5) (layer F.Cu) (net 6))
+  (segment (start 124.2 104.688222) (end 124.2 116.88) (width 1.5) (layer F.Cu) (net 6))
+  (segment (start 124.2 116.88) (end 126.7 119.38) (width 1.5) (layer F.Cu) (net 6))
+  (segment (start 128.327833 100.560389) (end 124.2 104.688222) (width 1.5) (layer F.Cu) (net 6))
+  (segment (start 141.580666 98.044) (end 139.064277 100.560389) (width 1.5) (layer F.Cu) (net 6))
   (segment (start 126.7 119.38) (end 127 119.38) (width 1.5) (layer F.Cu) (net 6))
   (segment (start 162.179 111.391) (end 162.179 110.812) (width 0.25) (layer F.Cu) (net 7))
@@
   (segment (start 148.209 121.92) (end 155.829 121.92) (width 1.5) (layer F.Cu) (net 10))
   (segment (start 155.829 119.38) (end 148.209 119.38) (width 1.5) (layer F.Cu) (net 11))
-  (segment (start 140.589 87.261) (end 140.589 86.761) (width 0.25) (layer F.Cu) (net 12))
-  (segment (start 140.589 86.761) (end 137.902 84.074) (width 0.25) (layer F.Cu) (net 12))
-  (segment (start 137.902 84.074) (end 137.16 84.074) (width 0.25) (layer F.Cu) (net 12))
-  (segment (start 132.08 97.028) (end 137.033 97.028) (width 5) (layer F.Cu) (net 12))
-  (segment (start 137.16 84.074) (end 137.795 84.074) (width 5) (layer F.Cu) (net 12))
-  (segment (start 137.795 84.074) (end 143.637 84.074) (width 5) (layer F.Cu) (net 12))
-  (segment (start 137.045 89.928) (end 137.16 84.074) (width 5) (layer F.Cu) (net 12))
-  (segment (start 137.073 96.988) (end 137.045 89.928) (width 5) (layer F.Cu) (net 12))
-  (segment (start 137.033 97.028) (end 137.073 96.988) (width 0.25) (layer F.Cu) (net 12))
+  (segment (start 132.08 96.988) (end 133.296002 96.988) (width 5) (layer F.Cu) (net 12))
+  (segment (start 133.296002 96.988) (end 137.438999 92.845003) (width 5) (layer F.Cu) (net 12))
+  (segment (start 137.438999 92.845003) (end 137.438999 86.350999) (width 5) (layer F.Cu) (net 12))
+  (segment (start 137.438999 86.350999) (end 139.802998 83.987) (width 5) (layer F.Cu) (net 12))
+  (segment (start 139.802998 83.987) (end 143.637 83.987) (width 5) (layer F.Cu) (net 12))
   (segment (start 138.18573 127) (end 144.3228 120.86293) (width 1.5) (layer F.Cu) (net 13))
   (segment (start 150.114 111.0548) (end 150.114 108.2548) (width 1.5) (layer F.Cu) (net 13))

Commit message: suggested changes
Routing:
- net Net-(P11-Pad2): track 20.7 -> 24.6 mm
Changed lines of the file:
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@@
     (links 32)
     (no_connects 0)
-    (area 113.74941 80.211999 183.252791 129.598203)
+    (area 113.74941 80.408997 183.252791 129.598203)
     (thickness 1.6)
     (drawings 13)
-    (tracks 88)
+    (tracks 91)
     (zones 0)
     (modules 23)
@@
     (add_net "Net-(D2-Pad2)")
     (add_net "Net-(D3-Pad2)")
+    (add_net "Net-(P11-Pad2)")
     (add_net "Net-(P3-Pad2)")
   )
@@
     (uvia_dia 0.3)
     (uvia_drill 0.1)
-    (add_net "Net-(P11-Pad2)")
   )
   (module Connectors_Molex:Molex_KK-6410-04_04x2.54mm_Straight (layer F.Cu)
@@
   (segment (start 148.209 121.92) (end 155.829 121.92) (width 1.5) (layer F.Cu) (net 10))
   (segment (start 155.829 119.38) (end 148.209 119.38) (width 1.5) (layer F.Cu) (net 11))
+  (segment (start 140.589 87.261) (end 140.589 86.761) (width 0.25) (layer F.Cu) (net 12))
+  (segment (start 140.589 86.761) (end 140.178999 86.350999) (width 0.25) (layer F.Cu) (net 12))
+  (segment (start 140.178999 86.350999) (end 137.438999 86.350999) (width 0.25) (layer F.Cu) (net 12))
   (segment (start 132.08 96.988) (end 133.296002 96.988) (width 5) (layer F.Cu) (net 12))
   (segment (start 133.296002 96.988) (end 137.438999 92.845003) (width 5) (layer F.Cu) (net 12))
