File: NANO_SLAVE_BOARD/NANO_SLAVE_BOARD.sch (KiCad schematic (older format))
At the start: 25 parts

Commit message: Nano Rev0.1
Parts:
- removed J? (x2): RJ12, symbol RJ12
- added J1: RJ45, Connect:RJ45_8, symbol RJ45
- P1, P2, P5: renamed from P?; footprint (none) -> ASSETS:10_PIN_IDC
- P3, P4: renamed from P?; footprint (none) -> ASSETS:S5B-PH-K-S(LF)(SN)
- R1, R10, R11, R12, R2, R3, R4, R5, R6, R7, R8, R9: renamed from R?; footprint (none) -> Resistors_SMD:R_0603
- U1: renamed from U?; footprint DIL20 -> ASSETS:ARDUINO_NANO
- gave numbers to parts that had none: 5
Connections:
- net S_Q7 is gone; now on net S_Q6: P5.5 (P5)
- net S_Q9 is gone; now on net S_SCK: P5.4 (P4)
- net +3V3: now also P5.7 (P7), J1.8; no longer P5.1 (P1)
- net +5V: now also P5.9 (P9); no longer P5.2 (P2)
- net A0: now also P1.7 (P7); no longer P1.3 (P3)
- net A2: now also P1.3 (P3); no longer P1.7 (P7)
- net D2: no longer Q5.3 (D), R12.2
- net D4: no longer P2.1 (P1)
- net D5: now also P2.6 (P6); no longer P2.4 (P4)
- net D6: now also P2.4 (P4); no longer P2.6 (P6)
- net D7: now also P1.6 (P6); no longer P1.1 (P1)
- net D9: now also Q5.3 (D), R12.2; no longer P1.6 (P6)
- net GND: now also J1.7, J1.9 (SHIELD)
- net S_CS: now also P5.2 (P2), J1.4; no longer P5.6 (P6)
- net S_MISO: now also J1.5
- net S_MOSI: now also P5.6 (P6), J1.6; no longer P5.7 (P7)
- net S_Q6: now also J1.2
- net S_Q8: now also J1.1
- net S_SCK: now also J1.3; no longer P5.9 (P9)

Commit message: rev0.1 complete
Parts:
- removed J1: RJ45, Connect:RJ45_8, symbol RJ45
- added J?: RJ45_SHIELDED, symbol RJ45_SHIELDED
Connections:
- net +3V3: now also J?.8
- net GND: now also J?.13 (SHIELD), J?.7
- net S_CS: now also J?.4
- net S_MISO: now also J?.5
- net S_MOSI: now also J?.6
- net S_Q6: now also J?.2
- net S_Q8: now also J?.1
- net S_SCK: now also J?.3
- no-connect marks 4 -> 9
Changed lines of the file:
@@
 	3800 5500 3900 5500
 Wire Wire Line
-	8400 1300 8650 1300
+	8350 1300 8650 1300
 Wire Wire Line
 	8650 1300 8650 1150
 Wire Wire Line
-	8400 1400 8850 1400
+	8350 1400 8850 1400
 Wire Wire Line
 	8850 1400 8850 1350
 Wire Wire Line
-	8400 1500 8850 1500
-Wire Wire Line
-	8400 1600 8700 1600
+	8350 1500 8850 1500
+Wire Wire Line
+	8350 1600 8700 1600
 Wire Wire Line
 	8700 1600 8700 1650
@@
 	8700 1650 8850 1650
 Wire Wire Line
-	8400 1700 8650 1700
+	8350 1700 8650 1700
 Wire Wire Line
 	8650 1700 8650 1800
@@
 Wire Wire Line
 	4900 4000 4900 4150
-$Comp
-L RJ45 J1
-U 1 1 59E2A119
-P 7950 1650
-F 0 "J1" H 8150 2150 50  0000 C CNN
-F 1 "RJ45" H 7800 2150 50  0000 C CNN
-F 2 "Connect:RJ45_8" H 7950 1650 50  0000 C CNN
-F 3 "" H 7950 1650 50  0000 C CNN
-	1    7950 1650
-	0    -1   -1   0
-$EndComp
-Wire Wire Line
-	8600 1800 8400 1800
+Wire Wire Line
+	8600 1800 8350 1800
 Text GLabel 8850 2250 2    60   Input ~ 0
 S_Q8
 Wire Wire Line
-	8400 1900 8550 1900
+	8350 1900 8550 1900
 Wire Wire Line
 	8550 1900 8550 2100
@@
 	8550 2100 8850 2100
 Wire Wire Line
-	8400 2000 8500 2000
+	8350 2000 8500 2000
 Wire Wire Line
 	8500 2000 8500 2250
@@
 $EndComp
 Wire Wire Line
-	7600 1100 7600 1050
+	7550 1100 7600 1050
 Wire Wire Line
 	7950 3850 8100 3850
@@
 Wire Wire Line
 	8900 3750 8900 3700
+$Comp
+L RJ45_SHIELDED J?
+U 1 1 59E4D6B3
+P 7900 1650
+F 0 "J?" H 8300 2150 50  0000 C CNN
+F 1 "RJ45_SHIELDED" V 7450 1700 50  0000 C CNN
+F 2 "" H 7900 1650 50  0000 C CNN
+F 3 "" H 7900 1650 50  0000 C CNN
+	1    7900 1650
+	0    -1   -1   0
+$EndComp
+NoConn ~ 7300 1950
+NoConn ~ 7300 1850
+NoConn ~ 7300 1450
+NoConn ~ 7300 1350
+NoConn ~ 2200 1250
 $EndSCHEMATC

Commit message: routing fixes
Parts:
- gave numbers to parts that had none: 1
Connections:
- net +3V3: now also J1.1; no longer J1.8
- net S_CS: now also J1.8; no longer J1.4
- net S_MISO: now also J1.2; no longer J1.5
- net S_MOSI: now also J1.4; no longer J1.6
- net S_Q6: now also J1.6; no longer J1.2
- net S_Q8: now also J1.5; no longer J1.1
Changed lines of the file:
@@
 L +3.3V #PWR010
 U 1 1 59DE4102
-P 8650 1150
-F 0 "#PWR010" H 8650 1000 50  0001 C CNN
-F 1 "+3.3V" H 8650 1290 50  0000 C CNN
-F 2 "" H 8650 1150 50  0000 C CNN
-F 3 "" H 8650 1150 50  0000 C CNN
-	1    8650 1150
-	1    0    0    -1
+P 8850 2400
+F 0 "#PWR010" H 8850 2250 50  0001 C CNN
+F 1 "+3.3V" H 8850 2540 50  0000 C CNN
+F 2 "" H 8850 2400 50  0000 C CNN
+F 3 "" H 8850 2400 50  0000 C CNN
+	1    8850 2400
+	0    1    1    0
 $EndComp
 $Comp
@@
 	-1   0    0    1
 $EndComp
-Text GLabel 8850 1500 2    60   Input ~ 0
+Text GLabel 8850 1800 2    60   Input ~ 0
 S_MOSI
-Text GLabel 8850 1650 2    60   Input ~ 0
+Text GLabel 8850 2100 2    60   Input ~ 0
 S_MISO
-Text GLabel 8850 1800 2    60   Input ~ 0
+Text GLabel 8650 1150 1    60   Input ~ 0
 S_CS
 Text GLabel 8850 1950 2    60   Input ~ 0
 S_SCK
-Text GLabel 8850 2100 2    60   Input ~ 0
+Text GLabel 8850 1500 2    60   Input ~ 0
 S_Q6
 $Comp
@@
 Wire Wire Line
 	8600 1800 8350 1800
-Text GLabel 8850 2250 2    60   Input ~ 0
+Text GLabel 8850 1650 2    60   Input ~ 0
 S_Q8
 Wire Wire Line
@@
 	8500 2000 8500 2250
 Wire Wire Line
-	8500 2250 8850 2250
+	8500 2250 8850 2400
 $Comp
 L GND #PWR028
@@
 	8900 3750 8900 3700
 $Comp
-L RJ45_SHIELDED J?
+L RJ45_SHIELDED J1
 U 1 1 59E4D6B3
 P 7900 1650
-F 0 "J?" H 8300 2150 50  0000 C CNN
+F 0 "J1" H 8300 2150 50  0000 C CNN
 F 1 "RJ45_SHIELDED" V 7450 1700 50  0000 C CNN
 F 2 "" H 7900 1650 50  0000 C CNN

Commit message: suggested changes
Connections:
- net S_Q6: now also P5.3 (P3); no longer P5.5 (P5)
- net S_Q8: now also P5.5 (P5); no longer P5.3 (P3)
Changed lines of the file:
@@
 	1    0    0    -1
 $EndComp
+Text GLabel 8750 4000 2    60   Input ~ 0
+S_Q6
 Text GLabel 8750 3850 2    60   Input ~ 0
-S_Q6
-Text GLabel 8750 4000 2    60   Input ~ 0
 S_Q8
 Wire Wire Line
